File: tps61500evm/tps61500evm.kicad_pcb (KiCad board)
At the start: 2 copper layers, 46 x 25 mm, 18 parts, among them J1 Vin, J2 PWM, J3 OVP_Resistor(R1), J4 EN_DIMC, J5 LEDs, J6 FB Resistor, U1 TPS61500PWPR

Commit message: Add files
Other:
- board text added: "GND"
- board text added: "Vout"
Changed lines of the file:
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@@
   (general
     (thickness 1.6)
-    (drawings 4)
+    (drawings 8)
     (tracks 102)
     (zones 0)
@@
       (padsonsilk false)
       (subtractmaskfromsilk false)
-      (outputformat 1)
+      (outputformat 4)
       (mirror false)
-      (drillshape 1)
+      (drillshape 0)
       (scaleselection 1)
-      (outputdirectory ""))
+      (outputdirectory "pdf/"))
   )
   (net 0 "")
@@
       (effects (font (size 1 1) (thickness 0.15)))
     )
-    (fp_text value LEDs (at 2.53 -4.9 270) (layer F.SilkS)
+    (fp_text value LEDs (at 2.2 -4.9 270) (layer F.SilkS)
       (effects (font (size 1 1) (thickness 0.15)))
     )
@@
       (effects (font (size 1 1) (thickness 0.15)))
     )
-    (fp_text value Vin (at 2.78 -4.72 90) (layer F.SilkS)
-      (effects (font (size 1 1) (thickness 0.15)))
+    (fp_text value Vin (at 5.5 -5 90) (layer F.SilkS)
+      (effects (font (size 1 1) (thickness 0.2)))
     )
     (fp_line (start 7.79 4) (end -2.71 4) (layer F.CrtYd) (width 0.05))
@@
       (effects (font (size 1 1) (thickness 0.15)))
     )
-    (fp_text value PWM (at 2.4 -4.7 270) (layer F.SilkS)
-      (effects (font (size 1 1) (thickness 0.15)))
+    (fp_text value PWM (at 5.2 -5 270) (layer F.SilkS)
+      (effects (font (size 1 1) (thickness 0.2)))
     )
     (fp_text user %R (at 2.54 0 90) (layer F.Fab)
@@
     )
   )
+  (gr_text GND (at 23.2 36.1 90) (layer F.SilkS)
+    (effects (font (size 1 1) (thickness 0.2)))
+  )
+  (gr_text GND (at 23.3 24.1 90) (layer F.SilkS)
+    (effects (font (size 1 1) (thickness 0.2)))
+  )
+  (gr_text GND (at 66.8 25.1 90) (layer F.SilkS)
+    (effects (font (size 0.5 0.5) (thickness 0.1)))
+  )
+  (gr_text Vout (at 66.8 17.5 90) (layer F.SilkS)
+    (effects (font (size 0.5 0.5) (thickness 0.1)))
+  )
   (gr_line (start 22 40) (end 22 15) (layer Edge.Cuts) (width 0.15))
   (gr_line (start 68 40) (end 22 40) (layer Edge.Cuts) (width 0.15))
   (gr_line (start 68 15) (end 68 40) (layer Edge.Cuts) (width 0.15))
   (gr_line (start 22 15) (end 68 15) (layer Edge.Cuts) (width 0.15))
-  (segment (start 48.9 23.9396) (end 48.9 24.6) (width 0.4) (layer F.Cu) (net 6))
   (segment (start 51.6 26.0214) (end 51.6 26.0214) (width 0.25) (layer F.Cu) (net 1))
   (segment (start 49.6656 27.9558) (end 51.6 26.0214) (width 0.25) (layer F.Cu) (net 1))
@@
   (segment (start 53.5344 25.3396) (end 53.2 25.674) (width 0.25) (layer F.Cu) (net 1))
   (segment (start 54.521 25.3396) (end 53.5344 25.3396) (width 0.25) (layer F.Cu) (net 1))
-  (via (at 56.1 28.9) (size 0.8) (drill 0.4) (layers F.Cu B.Cu) (net 4))
   (via (at 45.4 26.9) (size 0.8) (drill 0.4) (layers F.Cu B.Cu) (net 2))
   (segment (start 47.73912 26) (end 48.679 26) (width 0.25) (layer F.Cu) (net 2))
@@
   (segment (start 32.46 18.72) (end 34.79 21.05) (width 2) (layer F.Cu) (net 3))
   (segment (start 28.2 18.72) (end 32.46 18.72) (width 2) (layer F.Cu) (net 3))
+  (via (at 56.1 28.9) (size 0.8) (drill 0.4) (layers F.Cu B.Cu) (net 4))
   (segment (start 62.13 30.17) (end 62.1 30.2) (width 2) (layer F.Cu) (net 4))
   (segment (start 56.1 28.334315) (end 56.1 28.9) (width 0.25) (layer F.Cu) (net 4))
@@
   (segment (start 55.77 18.9) (end 55.59 19.08) (width 2) (layer F.Cu) (net 5))
   (segment (start 62.1 18.9) (end 55.77 18.9) (width 2) (layer F.Cu) (net 5))
+  (segment (start 48.9 23.9396) (end 48.9 24.6) (width 0.4) (layer F.Cu) (net 6))
   (segment (start 45.57 22.3) (end 48.79 19.08) (width 2) (layer F.Cu) (net 6))
   (segment (start 44.69 22.3) (end 45.57 22.3) (width 2) (layer F.Cu) (net 6))
