File: tps61500evm.sch (KiCad schematic (older format))
At the start: 18 parts, among them J1 Vin, J2 PWM, J3 OVP_Resistor(R1), J4 EN_DIMC, J5 LEDs, J6 Feedback Resistor, U1 TPS61500PWPR

Commit message: Updated files
Parts:
- C1, C2, C3, C4, C5, C6, C7: footprint Capacitor_SMD:C_0805_2012Metric -> lib_fp:C_0805_2012Metric
- D1: footprint Diode_SMD:D_SMC -> lib_fp:D_SMC
- J1, J2, J5, J6: footprint TerminalBlock:TerminalBlock_bornier-2_P5.08mm -> lib_fp:TerminalBlock_bornier-2_P5.08mm
- J3, J4: footprint Connector_PinHeader_2.54mm:PinHeader_1x02_P2.54mm_Vertical -> lib_fp:PinHeader_1x02_P2.54mm_Vertical
- L1: footprint Inductor_SMD:L_12x12mm_H8mm -> lib_fp:L_12x12mm_H8mm
- R2, R3: footprint Capacitor_SMD:C_0805_2012Metric -> lib_fp:R_0805_2012Metric
- U1: footprint TPS61500PWPR:SOP65P640X120-15N -> lib_fp:SOP65P640X120-15N
Changed lines of the file:
@@
 EESchema Schematic File Version 4
-LIBS:tps61500evm-cache
 EELAYER 26 0
 EELAYER END
@@
 F 0 "U1" H 5700 4820 50  0000 C CNN
 F 1 "TPS61500PWPR" H 5700 4729 50  0000 C CNN
-F 2 "TPS61500PWPR:SOP65P640X120-15N" H 5700 3850 50  0001 L BNN
+F 2 "lib_fp:SOP65P640X120-15N" H 5700 3850 50  0001 L BNN
 F 3 "HTSSOP-14 Texas Instruments" H 5700 3850 50  0001 L BNN
 F 4 "https://www.digikey.in/product-detail/en/texas-instruments/TPS61500PWPR/296-24014-1-ND/1985046?utm_source=snapeda&utm_medium=aggregator&utm_campaign=symbol" H 5700 3850 50  0001 L BNN "Field4"
@@
 F 0 "R3" V 6950 3600 50  0000 L CNN
 F 1 "33k" V 6850 3600 50  0000 L CNN
-F 2 "Capacitor_SMD:C_0805_2012Metric" V 6780 3650 50  0001 C CNN
+F 2 "lib_fp:R_0805_2012Metric" V 6780 3650 50  0001 C CNN
 F 3 "~" H 6850 3650 50  0001 C CNN
 	1    6850 3650
@@
 F 0 "R2" V 4150 4700 50  0000 L CNN
 F 1 "10k" V 4050 4650 50  0000 L CNN
-F 2 "Capacitor_SMD:C_0805_2012Metric" V 3980 4750 50  0001 C CNN
+F 2 "lib_fp:R_0805_2012Metric" V 3980 4750 50  0001 C CNN
 F 3 "~" H 4050 4750 50  0001 C CNN
 	1    4050 4750
@@
 F 0 "L1" V 5540 1950 50  0000 C CNN
 F 1 "15uH" V 5449 1950 50  0000 C CNN
-F 2 "Inductor_SMD:L_12x12mm_H8mm" H 5350 1950 50  0001 C CNN
+F 2 "lib_fp:L_12x12mm_H8mm" H 5350 1950 50  0001 C CNN
 F 3 "~" H 5350 1950 50  0001 C CNN
 	1    5350 1950
@@
 F 0 "C5" H 7115 4896 50  0000 L CNN
 F 1 "1uF" H 7115 4805 50  0000 L CNN
-F 2 "Capacitor_SMD:C_0805_2012Metric" H 7038 4700 50  0001 C CNN
+F 2 "lib_fp:C_0805_2012Metric" H 7038 4700 50  0001 C CNN
 F 3 "~" H 7000 4850 50  0001 C CNN
 	1    7000 4850
@@
 F 0 "C4" V 7300 3600 50  0000 L CNN
 F 1 "0.1uF" V 7600 3550 50  0000 L CNN
-F 2 "Capacitor_SMD:C_0805_2012Metric" H 7488 3500 50  0001 C CNN
+F 2 "lib_fp:C_0805_2012Metric" H 7488 3500 50  0001 C CNN
 F 3 "~" H 7450 3650 50  0001 C CNN
 	1    7450 3650
@@
 F 0 "C2" V 5800 2100 50  0000 L CNN
 F 1 "10uF" V 5900 2050 50  0000 L CNN
-F 2 "Capacitor_SMD:C_0805_2012Metric" H 6088 2000 50  0001 C CNN
+F 2 "lib_fp:C_0805_2012Metric" H 6088 2000 50  0001 C CNN
 F 3 "~" H 6050 2150 50  0001 C CNN
 	1    6050 2150
@@
 F 0 "C1" H 3850 2300 50  0000 L CNN
 F 1 "10uF" H 3850 2100 50  0000 L CNN
-F 2 "Capacitor_SMD:C_0805_2012Metric" H 3888 2050 50  0001 C CNN
+F 2 "lib_fp:C_0805_2012Metric" H 3888 2050 50  0001 C CNN
 F 3 "~" H 3850 2200 50  0001 C CNN
 	1    3850 2200
@@
 F 0 "C3" V 6350 3600 50  0000 L CNN
 F 1 "0.1uF" V 6650 3550 50  0000 L CNN
-F 2 "Capacitor_SMD:C_0805_2012Metric" H 6538 3500 50  0001 C CNN
+F 2 "lib_fp:C_0805_2012Metric" H 6538 3500 50  0001 C CNN
 F 3 "~" H 6500 3650 50  0001 C CNN
 	1    6500 3650
@@
 F 0 "D1" H 5750 1750 50  0000 L CNN
 F 1 "SS54" H 5700 1850 50  0000 L CNN
-F 2 "Diode_SMD:D_SMC" H 5800 1950 50  0001 C CNN
+F 2 "lib_fp:D_SMC" H 5800 1950 50  0001 C CNN
 F 3 "~" H 5800 1950 50  0001 C CNN
 	1    5800 1950
@@
 F 0 "J4" H 7250 4550 50  0000 R CNN
 F 1 "EN_DIMC" H 7250 4650 50  0000 R CNN
-F 2 "Connector_PinHeader_2.54mm:PinHeader_1x02_P2.54mm_Vertical" H 7300 4650 50  0001 C CNN
+F 2 "lib_fp:PinHeader_1x02_P2.54mm_Vertical" H 7300 4650 50  0001 C CNN
 F 3 "~" H 7300 4650 50  0001 C CNN
 	1    7300 4650
@@
 F 0 "C6" H 4250 2300 50  0000 L CNN
 F 1 "C" H 4250 2100 50  0000 L CNN
-F 2 "Capacitor_SMD:C_0805_2012Metric" H 4238 2050 50  0001 C CNN
+F 2 "lib_fp:C_0805_2012Metric" H 4238 2050 50  0001 C CNN
 F 3 "~" H 4200 2200 50  0001 C CNN
 	1    4200 2200
@@
 F 0 "C7" V 6550 2100 50  0000 L CNN
 F 1 "C" V 6650 2100 50  0000 L CNN
-F 2 "Capacitor_SMD:C_0805_2012Metric" H 6438 2000 50  0001 C CNN
+F 2 "lib_fp:C_0805_2012Metric" H 6438 2000 50  0001 C CNN
 F 3 "~" H 6400 2150 50  0001 C CNN
 	1    6400 2150
@@
 F 0 "J5" H 7529 1942 50  0000 L CNN
 F 1 "LEDs" H 7529 1851 50  0000 L CNN
-F 2 "TerminalBlock:TerminalBlock_bornier-2_P5.08mm" H 7450 1950 50  0001 C CNN
+F 2 "lib_fp:TerminalBlock_bornier-2_P5.08mm" H 7450 1950 50  0001 C CNN
 F 3 "~" H 7450 1950 50  0001 C CNN
 	1    7450 1950
@@
 F 0 "J6" H 7529 2392 50  0000 L CNN
 F 1 "Feedback Resistor" H 7529 2301 50  0000 L CNN
-F 2 "TerminalBlock:TerminalBlock_bornier-2_P5.08mm" H 7450 2400 50  0001 C CNN
+F 2 "lib_fp:TerminalBlock_bornier-2_P5.08mm" H 7450 2400 50  0001 C CNN
 F 3 "~" H 7450 2400 50  0001 C CNN
 	1    7450 2400
@@
 F 0 "J1" H 3500 2000 50  0000 C CNN
 F 1 "Vin" H 3500 2100 50  0000 C CNN
-F 2 "TerminalBlock:TerminalBlock_bornier-2_P5.08mm" H 3350 2100 50  0001 C CNN
+F 2 "lib_fp:TerminalBlock_bornier-2_P5.08mm" H 3350 2100 50  0001 C CNN
 F 3 "~" H 3350 2100 50  0001 C CNN
 	1    3350 2100
@@
 F 0 "J2" H 3750 3250 50  0000 C CNN
 F 1 "PWM" H 3750 3350 50  0000 C CNN
-F 2 "TerminalBlock:TerminalBlock_bornier-2_P5.08mm" H 3600 3350 50  0001 C CNN
+F 2 "lib_fp:TerminalBlock_bornier-2_P5.08mm" H 3600 3350 50  0001 C CNN
 F 3 "~" H 3600 3350 50  0001 C CNN
 	1    3600 3350
@@
 F 0 "J3" H 3750 4150 50  0000 C CNN
 F 1 "OVP_Resistor(R1)" H 4000 4250 50  0000 C CNN
-F 2 "Connector_PinHeader_2.54mm:PinHeader_1x02_P2.54mm_Vertical" H 3650 4250 50  0001 C CNN
+F 2 "lib_fp:PinHeader_1x02_P2.54mm_Vertical" H 3650 4250 50  0001 C CNN
 F 3 "~" H 3650 4250 50  0001 C CNN
 	1    3650 4250

Commit message: New 3d view
Parts:
- J3: footprint lib_fp:PinHeader_1x02_P2.54mm_Vertical -> Connector_PinSocket_2.54mm:PinSocket_1x02_P2.54mm_Vertical
Changed lines of the file:
@@
 EESchema Schematic File Version 4
+LIBS:tps61500evm-cache
 EELAYER 26 0
 EELAYER END
@@
 F 0 "J3" H 3750 4150 50  0000 C CNN
 F 1 "OVP_Resistor(R1)" H 4000 4250 50  0000 C CNN
-F 2 "lib_fp:PinHeader_1x02_P2.54mm_Vertical" H 3650 4250 50  0001 C CNN
+F 2 "Connector_PinSocket_2.54mm:PinSocket_1x02_P2.54mm_Vertical" H 3650 4250 50  0001 C CNN
 F 3 "~" H 3650 4250 50  0001 C CNN
 	1    3650 4250
